Commit message: added lidar, camera and depth camera

File: description/lidar.xacro (robot description, xacro)
@@ -1,137 +1,54 @@
 <?xml version="1.0"?>
 <robot xmlns:xacro="http://www.ros.org/wiki/xacro">
-   <xacro:property name="M_PI" value="3.1415926535897931" />
-  <xacro:macro name="VLP-16" params="*origin parent:=base_link name:=velodyne topic:=/velodyne_points hz:=10 lasers:=16 samples:=1875 collision_range:=0.8 min_range:=0.9 max_range:=130.0 noise:=0.008 min_angle:=-${M_PI} max_angle:=${M_PI} gpu:=false">
-    <joint name="lidar_joint" type="fixed">
-      <xacro:insert_block name="origin" />
-      <parent link="chassis_link"/>
-      <child link="lidar_link"/>
-    </joint>
-    <link name="lidar_link">
-      <inertial>
-        <mass value="0.83"/>
-        <origin xyz="0 0 0.03585"/>
-        <inertia ixx="${(0.83 * (3.0*0.0516*0.0516 + 0.0717*0.0717)) / 12.0}" ixy="0" ixz="0"
-          iyy="${(0.83 * (3.0*0.0516*0.0516 + 0.0717*0.0717)) / 12.0}" iyz="0"
-          izz="${0.5 * 0.83 * (0.0516*0.0516)}"/>
-      </inertial>
-      <visual>
-        <geometry>
-          <mesh filename="/meshes/VLP-16_base_1.dae" />
-        </geometry>
-      </visual>
-      <visual>
-        <geometry>
-          <mesh filename="/meshes/VLP-16_base_2.dae" />
-        </geometry>
-      </visual>
-      <collision>
-        <origin rpy="0 0 0" xyz="0 0 0.03585"/>
-        <geometry>
-          <cylinder radius="0.0516" length="0.0717"/>
-        </geometry>
-      </collision>
-    </link>
-    <joint name="lidar__top_joint" type="fixed" >
-      <origin xyz="0 0 0.0377" rpy="0 0 0" />
-      <parent link="lidar_link" />
-      <child link="top_link"/>
-    </joint>
-    <link name="top_link">
-      <inertial>
-        <mass value="0.01"/>
-        <origin xyz="0 0 0"/>
-        <inertia ixx="1e-7" ixy="0" ixz="0" iyy="1e-7" iyz="0" izz="1e-7"/>
-      </inertial>
-      <visual>
-        <origin xyz="0 0 -0.0377" />
-        <geometry>
-          <mesh filename="/meshes/VLP-16_scan.dae" />
-        </geometry>
-      </visual>
-    </link>
-    <!-- Gazebo requires the velodyne_gazebo_plugins package -->
-    <!-- <gazebo reference="${name}">
-      <xacro:if value="${gpu}">
-        <sensor type="gpu_ray" name="${name}-VLP16">
-          <pose>0 0 0 0 0 0</pose>
-          <visualize>false</visualize>
-          <update_rate>${hz}</update_rate>
-          <ray>
-            <scan>
-              <horizontal>
-                <samples>${samples}</samples>
-                <resolution>1</resolution>
-                <min_angle>${min_angle}</min_angle>
-                <max_angle>${max_angle}</max_angle>
-              </horizontal>
-              <vertical>
-                <samples>${lasers}</samples>
-                <resolution>1</resolution>
-                <min_angle>-${15.0*M_PI/180.0}</min_angle>
-                <max_angle> ${15.0*M_PI/180.0}</max_angle>
-              </vertical>
-            </scan>
-            <range>
-              <min>${collision_range}</min>
-              <max>${max_range+1}</max>
-              <resolution>0.001</resolution>
-            </range>
-            <noise>
-              <type>gaussian</type>
-              <mean>0.0</mean>
-              <stddev>0.0</stddev>
-            </noise>
-          </ray>
-          <plugin name="gazebo_ros_laser_controller" filename="libgazebo_ros_lidar_gpu.so">
-            <topicName>${topic}</topicName>
-            <frameName>${name}</frameName>
-            <min_range>${min_range}</min_range>
-            <max_range>${max_range}</max_range>
-            <gaussianNoise>${noise}</gaussianNoise>
-          </plugin>
+   <joint name="lidar_chassis_joint" type="fixed">
+    <parent link="chassis_link"/>
+    <child link="lidar_link"/>
+    <origin xyz="0.2 0.0 0.068" rpy="0.0 0.0 0.0"/>
+   </joint>
+  <link name="lidar_link">
+    <visual>
+    <geometry>
+      <cylinder radius="0.02" length="0.025"/>
+    </geometry>
+    <origin xyz="0.0 0.0 0.0125" rpy="0.0 0.0 0.0"/>
+    <material name="red" />
+    </visual>
+    <collision>
+      <geometry>
+        <cylinder radius="0.03375" length="0.025"/>
+      </geometry>
+      <origin xyz="0.0 0.0 0.0" rpy="0.0 0.0 0.0"/>
+    </collision>
+     <xacro:inertial_cylinder mass="0.5" radius="0.0675" length="0.025" >
+           <origin xyz="0.0 0.0 0.0" rpy="0.0 0.0 0.0"/>
+     </xacro:inertial_cylinder >
+  </link>
+  <gazebo reference="lidar_link">
+    <material>Gazebo/Red</material>
+    <sensor name="laser" type="ray">
+            <pose> 0 0 0 0 0 0 </pose>
+            <visualize>true</visualize>
+            <update_rate>10</update_rate>
+            <ray>
+                <scan>
+                    <horizontal>
+                        <samples>360</samples>
+                        <min_angle>-3.14</min_angle>
+                        <max_angle>3.14</max_angle>
+                    </horizontal>
+                </scan>
+                <range>
+                    <min>0.3</min>
+                    <max>12</max>
+                </range>
+            </ray>
+            <plugin name="laser_controller" filename="libgazebo_ros_ray_sensor.so">
+                <ros>
+                    <argument>~/out:=scan</argument>
+                </ros>
+                <output_type>sensor_msgs/LaserScan</output_type>
+                <frame_name>lidar_link</frame_name>
+            </plugin>
         </sensor>
-      </xacro:if>
-      <xacro:unless value="${gpu}">
-        <sensor type="ray" name="${name}-VLP16">
-          <pose>0 0 0 0 0 0</pose>
-          <visualize>false</visualize>
-          <update_rate>${hz}</update_rate>
-          <ray>
-            <scan>
-              <horizontal>
-                <samples>${samples}</samples>
-                <resolution>1</resolution>
-                <min_angle>${min_angle}</min_angle>
-                <max_angle>${max_angle}</max_angle>
-              </horizontal>
-              <vertical>
-                <samples>${lasers}</samples>
-                <resolution>1</resolution>
-                <min_angle>-${15.0*M_PI/180.0}</min_angle>
-                <max_angle> ${15.0*M_PI/180.0}</max_angle>
-              </vertical>
-            </scan>
-            <range>
-              <min>${collision_range}</min>
-              <max>${max_range+1}</max>
-              <resolution>0.001</resolution>
-            </range>
-            <noise>
-              <type>gaussian</type>
-              <mean>0.0</mean>
-              <stddev>0.0</stddev>
-            </noise>
-          </ray>
-          <plugin name="gazebo_ros_laser_controller" filename="libgazebo_ros_lidar.so">
-            <topicName>${topic}</topicName>
-            <frameName>${name}</frameName>
-            <min_range>${min_range}</min_range>
-            <max_range>${max_range}</max_range>
-            <gaussianNoise>${noise}</gaussianNoise>
-          </plugin>
-        </sensor>
-      </xacro:unless>
-    </gazebo> -->
-  </xacro:macro>
+  </gazebo>
 </robot>

File: description/robot.urdf.xacro (robot description, xacro)
@@ -3,3 +3,6 @@
   <xacro:include filename="gazebo_control.xacro"/>
   <xacro:include filename="robot_core.xacro"/>
+  <xacro:include filename="lidar.xacro"/>
+  <!-- <xacro:include filename="camera.xacro"/> -->
+  <xacro:include filename="depth_camera.xacro"/>
 </robot>

File: description/robot_core.xacro (robot description, xacro)
@@ -2,5 +2,4 @@
 <robot xmlns:xacro="http://www.ros.org/wiki/xacro">
   <xacro:include filename="inertial_macro.xacro"/>
-    <xacro:include filename="lidar.xacro"/>
  <material name="white">
     <color rgba=" 1 1 1 1" />
